Commit message: Fixed turning issue when follower loses the AR Tag

File: Harrison/catkin shit/turtlebot3/turtlebot3_description/urdf/turtlebot3_waffle_pi.gazebo.xacro (robot description, xacro)
@@ -17,4 +17,12 @@
     <material>Gazebo/FlatBlack</material>
   </gazebo>
+      <gazebo reference="simple_box_base_link">
+	<gravity> 0 </gravity>
+        <kp>100000.0</kp>
+        <kd>100000.0</kd>
+        <mu1>0.1</mu1>
+        <mu2>0.1</mu2>
+        <fdir>1 0 0</fdir>
+    </gazebo>
   <gazebo reference="wheel_right_link">
     <mu1>0.1</mu1>

File: Harrison/catkin shit/turtlebot3/turtlebot3_description/urdf/turtlebot3_waffle_pi.urdf.xacro (robot description, xacro)
@@ -31,4 +31,24 @@
     </inertial>
   </link>
+  <joint name="ar_tag_joint" type="fixed">
+    <parent link="base_footprint"/>
+    <child link="simple_box_base_link"/>
+    <origin xyz="-0.2 0.0 0.1" rpy="-1.57 3.14 1.57"/>
+    <axis xyz="0 0 1"/>
+  </joint>
+  <link name="simple_box_base_link">
+	<gravity> 0 </gravity>
+        <inertial>
+            <origin xyz="0 0 0" rpy="0 0 0"/>
+            <mass value="0.0001" />
+            <inertia ixx="0.0001" ixy="0.0" ixz="0.0" iyy="0.0001" iyz="0.0" izz="0.0001"/>
+        </inertial>
+        <visual>
+            <origin rpy="0.0 0 0" xyz="0 0 0"/>
+            <geometry>
+                <mesh filename="package://ar_tag_demo/meshes/ar_tag_0_to_3.dae"/>
+            </geometry>
+        </visual>
+    </link>
   <joint name="wheel_left_joint" type="continuous">
     <parent link="base_link"/>
